File: Hardware/LED-PCB/LED-PCB.kicad_pcb (KiCad board)
At the start: 2 copper layers, 200 x 200 mm, 225 parts, among them J1 Conn_01x03_Pin

Commit message: led placed
Parts:
- C1, C10, C100, C101, C102, C103, C104, C105, C106, C107, C108, C109, C11, C110, C12, C13, C14, C15, C16, C17, C18, C19, C2, C20, C21, C22, C23, C24, C25, C26, C27, C28, C29, C3, C30, C31, C32, C33, C34, C35, C36, C37, C38, C39, C4, C40, C41, C42, C43, C44, C45, C46, C47, C48, C49, C5, C50, C51, C52, C53, C54, C55, C56, C57, C58, C59, C6, C60, C61, C62, C63, C64, C65, C66, C67, C68, C69, C7, C70, C71, C72, C73, C74, C75, C76, C77, C78, C79, C8, C80, C81, C82, C83, C84, C85, C86, C87, C88, C89, C9, C90, C91, C92, C93, C94, C95, C96, C97, C98, C99: moved to B.Cu
- moved D100 326.4 mm to (66.7, 224.9)
- moved D89 311.0 mm to (66.7, 208.3), turned to 180 degrees
- moved D101 308.7 mm to (83.3, 224.9)
- moved D78 295.9 mm to (66.7, 191.6)
- moved D90 293.2 mm to (83.3, 208.3), turned to 180 degrees
- moved D102 291.1 mm to (100.0, 224.9)
- moved D67 281.3 mm to (66.7, 175.0), turned to 180 degrees
- moved D79 278.1 mm to (83.3, 191.6)
- moved D91 275.5 mm to (100.0, 208.3), turned to 180 degrees
- moved D103 273.5 mm to (116.6, 224.9)
- moved J1 269.5 mm to (58.5, 57.5)
- moved D56 267.1 mm to (66.7, 158.3)
- moved D68 263.4 mm to (83.3, 175.0), turned to 180 degrees
- moved D80 260.3 mm to (100.0, 191.6)
- moved D92 257.8 mm to (116.6, 208.3), turned to 180 degrees
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Connections:
- D100 pad 2: Net-(D100-DOUT) -> unconnected-(D100-DOUT-Pad2)
- D101 pad 2: Net-(D101-DOUT) -> Net-(D100-DIN)
- D101 pad 4: Net-(D100-DOUT) -> Net-(D101-DIN)
- D102 pad 2: Net-(D102-DOUT) -> Net-(D101-DIN)
- D102 pad 4: Net-(D101-DOUT) -> Net-(D102-DIN)
- D103 pad 2: Net-(D103-DOUT) -> Net-(D102-DIN)
- D103 pad 4: Net-(D102-DOUT) -> Net-(D103-DIN)
- D104 pad 2: Net-(D104-DOUT) -> Net-(D103-DIN)
- D104 pad 4: Net-(D103-DOUT) -> Net-(D104-DIN)
- D105 pad 2: Net-(D105-DOUT) -> Net-(D104-DIN)
- D105 pad 4: Net-(D104-DOUT) -> Net-(D105-DIN)
- D106 pad 2: Net-(D106-DOUT) -> Net-(D105-DIN)
- D106 pad 4: Net-(D105-DOUT) -> Net-(D106-DIN)
- D107 pad 2: Net-(D107-DOUT) -> Net-(D106-DIN)
- D107 pad 4: Net-(D106-DOUT) -> Net-(D107-DIN)
- D108 pad 2: Net-(D108-DOUT) -> Net-(D107-DIN)
- D108 pad 4: Net-(D107-DOUT) -> Net-(D108-DIN)
- D109 pad 2: Net-(D109-DOUT) -> Net-(D108-DIN)
- D109 pad 4: Net-(D108-DOUT) -> Net-(D109-DIN)
- D110 pad 2: unconnected-(D110-DOUT-Pad2) -> Net-(D109-DIN)
- D110 pad 4: Net-(D109-DOUT) -> Net-(D110-DIN)
- D12 pad 4: Net-(D11-DOUT) -> Net-(D12-DIN)
- D13 pad 2: Net-(D13-DOUT) -> Net-(D12-DIN)
- D13 pad 4: Net-(D12-DOUT) -> Net-(D13-DIN)
- D14 pad 2: Net-(D14-DOUT) -> Net-(D13-DIN)
- D14 pad 4: Net-(D13-DOUT) -> Net-(D14-DIN)
- D15 pad 2: Net-(D15-DOUT) -> Net-(D14-DIN)
- D15 pad 4: Net-(D14-DOUT) -> Net-(D15-DIN)
- D16 pad 2: Net-(D16-DOUT) -> Net-(D15-DIN)
- D16 pad 4: Net-(D15-DOUT) -> Net-(D16-DIN)
- D17 pad 2: Net-(D17-DOUT) -> Net-(D16-DIN)
- D17 pad 4: Net-(D16-DOUT) -> Net-(D17-DIN)
- D18 pad 2: Net-(D18-DOUT) -> Net-(D17-DIN)
- D18 pad 4: Net-(D17-DOUT) -> Net-(D18-DIN)
- D19 pad 2: Net-(D19-DOUT) -> Net-(D18-DIN)
- D19 pad 4: Net-(D18-DOUT) -> Net-(D19-DIN)
- D20 pad 2: Net-(D20-DOUT) -> Net-(D19-DIN)
- D20 pad 4: Net-(D19-DOUT) -> Net-(D20-DIN)
- D21 pad 2: Net-(D21-DOUT) -> Net-(D20-DIN)
- D21 pad 4: Net-(D20-DOUT) -> Net-(D21-DIN)
- D22 pad 2: Net-(D22-DOUT) -> Net-(D21-DIN)
- D22 pad 4: Net-(D21-DOUT) -> Net-(D11-DOUT)
- D23 pad 4: Net-(D22-DOUT) -> Net-(D12-DOUT)
- D34 pad 4: Net-(D33-DOUT) -> Net-(D34-DIN)
- D35 pad 2: Net-(D35-DOUT) -> Net-(D34-DIN)
- D35 pad 4: Net-(D34-DOUT) -> Net-(D35-DIN)
- D36 pad 2: Net-(D36-DOUT) -> Net-(D35-DIN)
- D36 pad 4: Net-(D35-DOUT) -> Net-(D36-DIN)
- D37 pad 2: Net-(D37-DOUT) -> Net-(D36-DIN)
- D37 pad 4: Net-(D36-DOUT) -> Net-(D37-DIN)
- D38 pad 2: Net-(D38-DOUT) -> Net-(D37-DIN)
- D38 pad 4: Net-(D37-DOUT) -> Net-(D38-DIN)
- D39 pad 2: Net-(D39-DOUT) -> Net-(D38-DIN)
- D39 pad 4: Net-(D38-DOUT) -> Net-(D39-DIN)
- D40 pad 2: Net-(D40-DOUT) -> Net-(D39-DIN)
- D40 pad 4: Net-(D39-DOUT) -> Net-(D40-DIN)
- D41 pad 2: Net-(D41-DOUT) -> Net-(D40-DIN)
- D41 pad 4: Net-(D40-DOUT) -> Net-(D41-DIN)
- D42 pad 2: Net-(D42-DOUT) -> Net-(D41-DIN)
- D42 pad 4: Net-(D41-DOUT) -> Net-(D42-DIN)
- D43 pad 2: Net-(D43-DOUT) -> Net-(D42-DIN)
- D43 pad 4: Net-(D42-DOUT) -> Net-(D43-DIN)
- D44 pad 2: Net-(D44-DOUT) -> Net-(D43-DIN)
- D44 pad 4: Net-(D43-DOUT) -> Net-(D33-DOUT)
- D45 pad 4: Net-(D44-DOUT) -> Net-(D34-DOUT)
- D56 pad 4: Net-(D55-DOUT) -> Net-(D56-DIN)
- D57 pad 2: Net-(D57-DOUT) -> Net-(D56-DIN)
- D57 pad 4: Net-(D56-DOUT) -> Net-(D57-DIN)
- D58 pad 2: Net-(D58-DOUT) -> Net-(D57-DIN)
- D58 pad 4: Net-(D57-DOUT) -> Net-(D58-DIN)
- D59 pad 2: Net-(D59-DOUT) -> Net-(D58-DIN)
- D59 pad 4: Net-(D58-DOUT) -> Net-(D59-DIN)
- D60 pad 2: Net-(D60-DOUT) -> Net-(D59-DIN)
- D60 pad 4: Net-(D59-DOUT) -> Net-(D60-DIN)
- D61 pad 2: Net-(D61-DOUT) -> Net-(D60-DIN)
- D61 pad 4: Net-(D60-DOUT) -> Net-(D61-DIN)
- D62 pad 2: Net-(D62-DOUT) -> Net-(D61-DIN)
- D62 pad 4: Net-(D61-DOUT) -> Net-(D62-DIN)
- D63 pad 2: Net-(D63-DOUT) -> Net-(D62-DIN)
- D63 pad 4: Net-(D62-DOUT) -> Net-(D63-DIN)
- D64 pad 2: Net-(D64-DOUT) -> Net-(D63-DIN)
- D64 pad 4: Net-(D63-DOUT) -> Net-(D64-DIN)
- D65 pad 2: Net-(D65-DOUT) -> Net-(D64-DIN)
- D65 pad 4: Net-(D64-DOUT) -> Net-(D65-DIN)
- D66 pad 2: Net-(D66-DOUT) -> Net-(D65-DIN)
- D66 pad 4: Net-(D65-DOUT) -> Net-(D55-DOUT)
- D67 pad 4: Net-(D66-DOUT) -> Net-(D56-DOUT)
- D78 pad 4: Net-(D77-DOUT) -> Net-(D78-DIN)
- D79 pad 2: Net-(D79-DOUT) -> Net-(D78-DIN)
- D79 pad 4: Net-(D78-DOUT) -> Net-(D79-DIN)
- D80 pad 2: Net-(D80-DOUT) -> Net-(D79-DIN)
- D80 pad 4: Net-(D79-DOUT) -> Net-(D80-DIN)
- D81 pad 2: Net-(D81-DOUT) -> Net-(D80-DIN)
- D81 pad 4: Net-(D80-DOUT) -> Net-(D81-DIN)
- D82 pad 2: Net-(D82-DOUT) -> Net-(D81-DIN)
- D82 pad 4: Net-(D81-DOUT) -> Net-(D82-DIN)
- D83 pad 2: Net-(D83-DOUT) -> Net-(D82-DIN)
- D83 pad 4: Net-(D82-DOUT) -> Net-(D83-DIN)
- D84 pad 2: Net-(D84-DOUT) -> Net-(D83-DIN)
- D84 pad 4: Net-(D83-DOUT) -> Net-(D84-DIN)
- D85 pad 2: Net-(D85-DOUT) -> Net-(D84-DIN)
- D85 pad 4: Net-(D84-DOUT) -> Net-(D85-DIN)
- D86 pad 2: Net-(D86-DOUT) -> Net-(D85-DIN)
- D86 pad 4: Net-(D85-DOUT) -> Net-(D86-DIN)
- D87 pad 2: Net-(D87-DOUT) -> Net-(D86-DIN)
- D87 pad 4: Net-(D86-DOUT) -> Net-(D87-DIN)
- D88 pad 2: Net-(D88-DOUT) -> Net-(D87-DIN)
- D88 pad 4: Net-(D87-DOUT) -> Net-(D77-DOUT)
- D89 pad 4: Net-(D88-DOUT) -> Net-(D78-DOUT)
- D99 pad 2: Net-(D100-DIN) -> Net-(D110-DIN)
Routing:
- net +5V: track 0.00 -> 485.4 mm, vias 0 -> 21
- net Net-(D56-DOUT): track 0.00 -> 17.6 mm
- net Net-(D78-DOUT): track 0.00 -> 17.6 mm
- net Net-(D12-DOUT): track 0.00 -> 17.6 mm
- net Net-(D34-DOUT): track 0.00 -> 17.6 mm
- net Net-(D11-DOUT): track 0.00 -> 17.6 mm
- net Net-(D77-DOUT): track 0.00 -> 17.6 mm
- net Net-(D110-DIN): track 0.00 -> 17.6 mm
- net Net-(D55-DOUT): track 0.00 -> 17.6 mm
- net Net-(D33-DOUT): track 0.00 -> 17.6 mm
- net Net-(D97-DOUT): track 0.00 -> 13.1 mm
- net Net-(D96-DOUT): track 0.00 -> 13.1 mm
- net Net-(D95-DOUT): track 0.00 -> 13.1 mm
- net Net-(D86-DIN): track 0.00 -> 13.1 mm
- net Net-(D85-DIN): track 0.00 -> 13.1 mm
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- removed copper zone on B.Cu, net GND

Commit message: placed capacitors
Parts:
- moved C100 212.6 mm to (66.7, 224.9), turned to 0 degrees
- moved C89 206.8 mm to (66.7, 208.3)
- moved C67 205.0 mm to (66.7, 175.0)
- moved C78 204.2 mm to (66.7, 191.6), turned to 0 degrees
- moved C101 196.4 mm to (83.3, 224.9), turned to 0 degrees
- moved C90 190.1 mm to (83.3, 208.3)
- moved C68 188.1 mm to (83.3, 175.0)
- moved C79 187.3 mm to (83.3, 191.6), turned to 0 degrees
- moved C102 180.4 mm to (100.0, 224.9), turned to 0 degrees
- moved C91 173.5 mm to (100.0, 208.3)
- moved C69 171.3 mm to (100.0, 175.0)
- moved C80 170.4 mm to (100.0, 191.6), turned to 0 degrees
- moved C103 164.6 mm to (116.6, 224.9), turned to 0 degrees
- moved C92 157.0 mm to (116.6, 208.3)
- moved C70 154.5 mm to (116.6, 175.0)
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Routing:
- net +5V: track 485.4 -> 2607.0 mm, vias 21 -> 109

Commit message: add gnd vias
Connections:
- C12 pad 2: Net-(C12-Pad2) -> GND
- C13 pad 2: Net-(C12-Pad2) -> GND
- C14 pad 2: Net-(C12-Pad2) -> GND
- C15 pad 2: Net-(C12-Pad2) -> GND
- C16 pad 2: Net-(C12-Pad2) -> GND
- C17 pad 2: Net-(C12-Pad2) -> GND
- C18 pad 2: Net-(C12-Pad2) -> GND
- C19 pad 2: Net-(C12-Pad2) -> GND
- C20 pad 2: Net-(C12-Pad2) -> GND
- C21 pad 2: Net-(C12-Pad2) -> GND
- C22 pad 2: Net-(C12-Pad2) -> GND
Routing:
- net +5V: track 2607.0 -> 2610.0 mm, vias 109 -> 110
- net GND: vias 0 -> 220
- added copper zone on B.Cu, net GND

Commit message: change connector and place mounting holes
Parts:
- added H5: MountingHole, MountingHole:MountingHole_3.2mm_M3, F.Cu at (66.7, 60.0)
- added H6: MountingHole, MountingHole:MountingHole_3.2mm_M3, F.Cu at (233.3, 60.0)
- added H7: MountingHole, MountingHole:MountingHole_3.2mm_M3, F.Cu at (66.7, 239.9)
- added H8: MountingHole, MountingHole:MountingHole_3.2mm_M3, F.Cu at (233.3, 239.9)
- J1: footprint Connector_JST:JST_XH_B3B-XH-AM_1x03_P2.50mm_Vertical -> lib:HDR-SMD_3P-P2.54-H-M_KH-2.54PH-1X3P-L13.5-WT; moved to B.Cu
- moved H3 324.9 mm to (56.7, 232.9)
- moved H1 304.6 mm to (56.7, 67.0)
- moved H4 159.8 mm to (243.3, 232.9)
- moved H2 123.1 mm to (243.3, 67.0)
- moved J1 25.3 mm to (83.6, 61.0), turned to -90 degrees
Routing:
- net /DATA: track 0.00 -> 31.9 mm, vias 0 -> 1
- net +5V: track 2610.0 -> 2626.5 mm
- net GND: vias 220 -> 500
Other:
- board text added: "LED-PCB @casartar 2025"
